File: Hardware/Vexus PCB V2/kicad de prueba.kicad_pcb (KiCad board)
At the start: 2 copper layers, 110 x 50 mm, 57 parts, among them J1 Conn_01x02_Pin, J10 Conn_01x04_Pin, J11 Conn_01x03_Pin, J12 Conn_01x03_Pin, J13 Conn_01x03_Pin, J14 Conn_01x03_Pin, J15 Conn_01x03_Pin, J16 Conn_01x04_Pin, J18 Conn_01x04_Pin, J19 Conn_01x04_Pin, J2 Conn_01x02_Pin, J3 Conn_01x03_Pin, J4 BTS-1, J5 BTS-2, J6 Conn_01x03_Pin, J7 Conn_01x03_Pin, J8 Conn_01x03_Pin, J9 Conn_01x10_Pin, SW1 SW_DPST_x2, SW5 SW_Push_Dual_x2, SW6 SW_Push_Dual_x2, SW7 SW_Push_Dual_x2, SW8 SW_Push_Dual_x2, SW9 SW_Push_Dual_x2, U1 ESP32-S3-WROOM-1, U2 AMS1117-3.3, U3 24LC64, U4 4051

Commit message: Add files via upload
Parts:
- added C10: 100nF, Capacitor_SMD:C_0805_2012Metric_Pad1.18x1.45mm_HandSolder, F.Cu at (176.8, 79.8)
- added C8: 100nF, Capacitor_SMD:C_0805_2012Metric_Pad1.18x1.45mm_HandSolder, F.Cu at (190.7, 79.8)
- added C9: 100nF, Capacitor_SMD:C_0805_2012Metric_Pad1.18x1.45mm_HandSolder, F.Cu at (183.8, 79.8)
- added J17: Conn_01x02_Pin, Connector_JST:JST_XH_B2B-XH-A_1x02_P2.50mm_Vertical, F.Cu at (175.8, 90.2)
- added R25: 1K, Resistor_SMD:R_0805_2012Metric_Pad1.20x1.40mm_HandSolder, F.Cu at (173.2, 100.0)
- added R26: 1K, Resistor_SMD:R_0805_2012Metric_Pad1.20x1.40mm_HandSolder, F.Cu at (175.2, 100.0)
- R10: value 10k -> 1k
- moved R20 4.50 mm to (172.2, 108.8), turned to 0 degrees
- moved U3 3.31 mm to (185.6, 104.1)
- moved R19 3.25 mm to (168.5, 108.8)
- moved R22 2.70 mm to (130.8, 106.0)
- moved R15 2.50 mm to (111.0, 108.8), turned to 180 degrees
- moved R21 2.50 mm to (130.8, 108.2), turned to 180 degrees
- moved D1 2.30 mm to (193.2, 97.5)
- moved R1 2.30 mm to (190.2, 97.5)
- moved R23 2.00 mm to (194.0, 104.2)
- moved R24 2.00 mm to (192.0, 104.2), turned to -90 degrees
- moved R17 1.50 mm to (111.0, 106.8)
- moved R18 1.03 mm to (177.8, 109.0)
- moved J8 1.00 mm to (171.5, 74.8)
- moved C3 0.81 mm to (122.0, 81.0)
- moved R16 0.35 mm to (183.0, 109.0), turned to 180 degrees
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Connections:
- R16 pad 2: /S4 -> /S2
- R17 pad 1: Net-(J12-Pin_2) -> /S5
- R18 pad 1: Net-(J15-Pin_2) -> /S2
- R20 pad 1: Net-(J14-Pin_2) -> /S3
- R21 pad 2: /S1 -> /S4
- R22 pad 1: Net-(J11-Pin_2) -> /S4
- R23 pad 2: /S2 -> /S1
- R24 pad 1: Net-(J13-Pin_2) -> /S1
- U1 pad 18: unconnected-(U1-IO10-Pad18) -> /S3
- U1 pad 19: unconnected-(U1-IO11-Pad19) -> /S2
- U1 pad 20: unconnected-(U1-IO12-Pad20) -> /OUT2
- U1 pad 21: unconnected-(U1-IO13-Pad21) -> /OUT1
- U1 pad 22: /S3 -> unconnected-(U1-IO14-Pad22)
- U1 pad 23: /T2 -> unconnected-(U1-IO21-Pad23)
- U1 pad 24: /T3 -> unconnected-(U1-IO47-Pad24)
- U1 pad 38: /S2 -> /S1
- U1 pad 39: /S4 -> /T3
- U1 pad 8: /S1 -> /S4
Routing:
- net /T2: track 57.3 -> 0.00 mm
- net /OUT2: track 0.00 -> 42.1 mm, vias 0 -> 1
- net /OUT1: track 0.00 -> 28.4 mm, vias 0 -> 1
- net /S4: track 59.8 -> 37.1 mm, vias 2 -> 0
- net /S1: track 35.9 -> 55.8 mm, vias 0 -> 2
- net /S2: track 52.1 -> 68.6 mm, vias 2 -> 0
- net /T3: track 29.4 -> 13.8 mm, vias 1 -> 0
- net +3.3V: track 62.3 -> 76.8 mm
- net /S3: track 60.8 -> 75.2 mm
- net /SDA: track 51.9 -> 61.9 mm
- net /SCL: track 65.7 -> 73.0 mm
- net /L1: track 34.2 -> 39.2 mm
- net /S5: track 52.0 -> 55.3 mm
- net GND: track 2.24 -> 4.85 mm, vias 8 -> 9
- net +5V: track 57.3 -> 59.8 mm, vias 1 -> 2
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Other:
- board text removed: "FACU"
- board text removed: "RAMI"
- board text removed: "ULI"

Commit message: Add files via upload
Parts:
- added C11: 100nF, Capacitor_SMD:C_0805_2012Metric_Pad1.18x1.45mm_HandSolder, F.Cu at (170.5, 90.5)
- added C12: 100nF, Capacitor_SMD:C_0805_2012Metric_Pad1.18x1.45mm_HandSolder, F.Cu at (186.8, 91.2)
- added R8: 10k, Resistor_SMD:R_0805_2012Metric_Pad1.20x1.40mm_HandSolder, F.Cu at (172.7, 90.5)
- added R9: 10k, Resistor_SMD:R_0805_2012Metric_Pad1.20x1.40mm_HandSolder, F.Cu at (184.5, 91.2)
- moved J17 4.50 mm to (180.2, 90.2)
Connections:
- J16 pad 3: /SCL -> /SCL2
- J16 pad 4: /SDA -> /SDA2
- J17 pad 1: /OUT2 -> Net-(J17-Pin_1)
- J17 pad 2: /OUT1 -> Net-(J17-Pin_2)
- U1 pad 12: /SDA -> /B
- U1 pad 13: /B -> /C
- U1 pad 14: /C -> /SIG
- U1 pad 15: /SIG -> /SCL2
- U1 pad 17: /SCL -> /SDA
- U1 pad 18: /S3 -> /SCL
- U1 pad 19: /S2 -> /S3
- U1 pad 20: /OUT2 -> /S2
- U1 pad 21: /OUT1 -> /OUT2
- U1 pad 22: unconnected-(U1-IO14-Pad22) -> /OUT1
- U1 pad 23: unconnected-(U1-IO21-Pad23) -> /SDA2
Routing:
- net /SDA2: track 0.00 -> 45.9 mm, vias 0 -> 1
- net /SCL2: track 0.00 -> 21.8 mm, vias 0 -> 1
- net /SDA: track 61.9 -> 47.2 mm
- net Net-(J17-Pin_1): track 0.00 -> 10.1 mm, vias 0 -> 1
- net Net-(J17-Pin_2): track 0.00 -> 9.02 mm, vias 0 -> 1
- net /SCL: track 73.0 -> 65.1 mm
- net /OUT1: track 28.4 -> 22.1 mm, vias 1 -> 0
- net /C: track 9.61 -> 14.0 mm
- net /OUT2: track 42.1 -> 38.1 mm, vias 1 -> 0
- net GND: track 4.85 -> 8.54 mm, vias 9 -> 11
- net /B: track 14.9 -> 18.4 mm
- net /SIG: track 13.6 -> 16.9 mm
- net /S2: track 68.6 -> 66.6 mm
- net /S3: track 75.2 -> 73.4 mm
- net /TXD: track 20.7 -> 21.2 mm

Commit message: Add files via upload
Parts:
- R1: value R_Small -> 220
Connections:
- U1 pad 17: /SDA -> /SCL
- U1 pad 18: /SCL -> /SDA
- U1 pad 26: unconnected-(U1-IO45-Pad26) -> /T2
Routing:
- net /T2: track 0.00 -> 61.3 mm, vias 0 -> 2
- net /SCL: track 65.1 -> 43.8 mm
- net /SDA: track 47.2 -> 43.8 mm
- net Net-(J17-Pin_1): track 10.1 -> 7.26 mm
- net /BT: track 76.7 -> 74.8 mm
