File: Hardware/Vexus PCB V2/kicad de prueba.kicad_sch (KiCad schematic)
At the start: 58 parts, among them J1 Conn_01x02_Pin, J10 Conn_01x04_Pin, J11 Conn_01x03_Pin, J12 Conn_01x03_Pin, J13 Conn_01x03_Pin, J14 Conn_01x03_Pin, J15 Conn_01x03_Pin, J16 Conn_01x04_Pin, J17 Conn_01x04_Pin, J18 Conn_01x04_Pin, J19 Conn_01x04_Pin, J2 Conn_01x02_Pin, J3 Conn_01x03_Pin, J4 BTS-1, J5 BTS-2, J6 Conn_01x03_Pin, J7 Conn_01x03_Pin, J8 Conn_01x03_Pin, J9 Conn_01x10_Pin, SW1 SW_DPST_x2, SW5 SW_Push_Dual_x2, SW6 SW_Push_Dual_x2, SW7 SW_Push_Dual_x2, SW8 SW_Push_Dual_x2, SW9 SW_Push_Dual_x2, U1 ESP32-S3-WROOM-1, U2 AMS1117-3.3, U3 24LC64, U4 4051

Commit message: Add files via upload
Parts:
- removed J17: Conn_01x04_Pin, symbol Connector:Conn_01x04_Pin
- added C10, C8, C9: 100nF, Capacitor_SMD:C_0805_2012Metric_Pad1.18x1.45mm_HandSolder, symbol Device:C_Small
- added J17: Conn_01x02_Pin, Connector_JST:JST_XH_B2B-XH-A_1x02_P2.50mm_Vertical, symbol Connector:Conn_01x02_Pin
- added R25, R26: 1K, Resistor_SMD:R_0805_2012Metric_Pad1.20x1.40mm_HandSolder, symbol 2019---Sumo---NANO---BTS7960-rescue:R-EESTN5
- R10: value 10k -> 1k
Connections:
- net +3.3V: now also R25.2, R26.2
- net GND: now also C10.2, C8.2, C9.2
- net S1: now also R23.2, R24.1, U1.38 (IO2); no longer R21.2, U1.8 (IO15)
- net S2: now also R16.2, R18.1, U1.19 (IO11); no longer R23.2, U1.38 (IO2)
- net S3: now also R20.1, U1.18 (IO10); no longer U1.22 (IO14)
- net S4: now also R21.2, R22.1, U1.8 (IO15); no longer R16.2, U1.39 (IO1)
- net S5: now also R17.1
- net SCL: now also R26.1
- net SDA: now also R25.1
- net SW1: now also C10.1
- net SW2: now also C9.1
- net SW3: now also C8.1
- net T2: no longer U1.23 (IO21)
- net T3: now also U1.39 (IO1); no longer U1.24 (IO47)
- net at J15.2 (Pin_2), R16.1: no longer R18.1
- net at J13.2 (Pin_2), R23.1: no longer R24.1
- net at J11.2 (Pin_2), R21.1: no longer R22.1
- net OUT2: now reaches U1.20 (IO12)
- net OUT2: now also J17.1 (Pin_1)
- net OUT1: now reaches U1.21 (IO13)
- net OUT1: now also J17.2 (Pin_2)
- net at J12.2 (Pin_2), R15.1: no longer R17.1
- net at J14.2 (Pin_2), R19.1: no longer R20.1
Other:
- moved on the sheet: D1, J2, R1, R3, R4, R5, SW7A, SW8A, SW9A

Commit message: Add files via upload
Parts:
- added C11, C12: 100nF, Capacitor_SMD:C_0805_2012Metric_Pad1.18x1.45mm_HandSolder, symbol Device:C_Small
- added R8, R9: 10k, Resistor_SMD:R_0805_2012Metric_Pad1.20x1.40mm_HandSolder, symbol EESTN5:R
Connections:
- net B: now also U1.12 (IO8); no longer U1.13 (USB_D-)
- net C: now also U1.13 (USB_D-); no longer U1.14 (USB_D+)
- net GND: now also C11.1, C12.1
- net OUT1: now also U1.22 (IO14), C11.2, R8.2; no longer J17.2 (Pin_2), U1.21 (IO13)
- net OUT2: now also U1.21 (IO13), C12.2, R9.2; no longer J17.1 (Pin_1), U1.20 (IO12)
- net S2: now also U1.20 (IO12); no longer U1.19 (IO11)
- net S3: now also U1.19 (IO11); no longer U1.18 (IO10)
- net SCL: now also U1.18 (IO10); no longer J16.3 (Pin_3), U1.17 (IO9)
- net SDA: now also U1.17 (IO9); no longer J16.4 (Pin_4), U1.12 (IO8)
- net SIG: now also U1.14 (USB_D+); no longer U1.15 (IO3)
- net SDA2: now reaches U1.23 (IO21)
- net SDA2: now also J16.4 (Pin_4)
- new net: J17.2 (Pin_2), R8.1
- new net: J17.1 (Pin_1), R9.1
- new net SCL2: J16.3 (Pin_3), U1.15 (IO3)
Other:
- moved on the sheet: J17

Commit message: Add files via upload
Parts:
- R1: value R_Small -> 220
Connections:
- net SCL: now also U1.17 (IO9); no longer U1.18 (IO10)
- net SDA: now also U1.18 (IO10); no longer U1.17 (IO9)
- net T2: now also U1.26 (IO45)
- no-connect marks 7 -> 6
Other:
- note added: "DISPLAY OLED"
- note added: "DRIVERS BTS7960"
- note added: "EEPROM"
- note added: "ENCODERS"
- note added: "LED INDICATIVO"
- note added: "MODULO RELÉ"
- note added: "MULTIPLEXOR"
- note added: "REGLETA QTR8A"
- note added: "SENSORES SHARPS"
- note added: "SENSORES TCRT5000"
- title: (none) -> TRIATLON PCB "VEXUS"
- moved on the sheet: C1, C3, C4, C7, D1, J1, J10, J14, J15, J16, J17, J18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
